Commit message: 自主巡航：信号灯停车、定位修复与入口统一，实验产物不再入库
感知与控制
- 前向障碍检测改为按车身完整轮廓（含转弯时车尾扫掠）计算扫掠走廊，
  并逐扇区校验激光可见性，盲区直接判为不可通行。
- 局部 ICP 增加 ±6 cm 有界平移粗搜索与 Cauchy 权重，修复在重复表面
  （A 弯下坡）收敛到错误位姿导致的定位发散；新增真实扫描回归夹具
  test/fixtures/a_bend_scan.npz。

信号灯与停车
- 红灯、黄灯或灯色不可确认时，在本方向停车线前停车等待；绿灯需连续
  3 个新图像帧确认后起步，/autonomy/status.reason 区分等待与确认中。
- 只有实际车头越线才锁存 CROSSING，越线后完成驶离。

入口与默认参数
- 自主入口统一为 launch_car.sh --autonomy，launch_autonomy.sh 成为同一
  入口的快捷方式；GUI 使用 X11/Ogre1，仅传感器服务器使用 Ogre2。
- 默认速度提升至 0.15 m/s，弯道/坡道降至 0.09 m/s，车道无效降至 0.05。

仓库清理
- reports/autonomy/ 下的运行产物（逐次运行的 JSON 转储、启动日志、探针
  数据与截图）移出版本控制并加入 .gitignore，仅保留手写 markdown 报告。
  产物文件仍保留在本地工作区。

Co-Authored-By: Claude Code <noreply@anthropic.com>

File: src/dongfeng_description/urdf/dongfeng_car.urdf.xacro (robot description, xacro)
@@ -1,5 +1,5 @@
 <?xml version='1.0' encoding='utf-8'?>
 <robot name="dongfeng_car">
-  <!--Generated by scripts/generate_vehicle.py. X forward, Y left, Z up. File keeps the .xacro name for launch compatibility. Sensors are geometry/frames only.-->
+  <!--Generated by scripts/generate_vehicle.py. X forward, Y left, Z up. Camera, lidar and IMU publish through Gazebo Sensors.-->
   <link name="base_link">
     <visual name="base_shell">
@@ -169,5 +169,5 @@
       </material>
     </visual>
-    <collision name="rolling_tyre">
+    <collision>
       <origin xyz="0 0 0" rpy="-1.57079633 0 0" />
       <geometry>
@@ -192,4 +192,5 @@
     <kp>1000000</kp>
     <kd>100</kd>
+    <fdir1>0 0 1</fdir1>
   </gazebo>
   <link name="wheel_left_front_link">
@@ -221,5 +222,5 @@
       </material>
     </visual>
-    <collision name="rolling_tyre">
+    <collision>
       <origin xyz="0 0 0" rpy="-1.57079633 0 0" />
       <geometry>
@@ -244,4 +245,5 @@
     <kp>1000000</kp>
     <kd>100</kd>
+    <fdir1>0 0 1</fdir1>
   </gazebo>
   <link name="wheel_right_link">
@@ -273,5 +275,5 @@
       </material>
     </visual>
-    <collision name="rolling_tyre">
+    <collision>
       <origin xyz="0 0 0" rpy="-1.57079633 0 0" />
       <geometry>
@@ -296,4 +298,5 @@
     <kp>1000000</kp>
     <kd>100</kd>
+    <fdir1>0 0 1</fdir1>
   </gazebo>
   <link name="wheel_right_front_link">
@@ -325,5 +328,5 @@
       </material>
     </visual>
-    <collision name="rolling_tyre">
+    <collision>
       <origin xyz="0 0 0" rpy="-1.57079633 0 0" />
       <geometry>
@@ -348,4 +351,5 @@
     <kp>1000000</kp>
     <kd>100</kd>
+    <fdir1>0 0 1</fdir1>
   </gazebo>
   <link name="lidar_link">
@@ -472,4 +476,59 @@
     <origin xyz="0.0015 0 0" rpy="-1.57079633 0 -1.57079633" />
   </joint>
+  <gazebo reference="camera_link">
+    <sensor name="front_camera" type="camera">
+      <pose>0.007 0 0 0 0 0</pose>
+      <topic>/camera/image_raw</topic>
+      <always_on>true</always_on>
+      <update_rate>20</update_rate>
+      <gz_frame_id>camera_optical_frame</gz_frame_id>
+      <camera>
+        <horizontal_fov>1.8</horizontal_fov>
+        <image>
+          <width>640</width>
+          <height>480</height>
+          <format>R8G8B8</format>
+        </image>
+        <clip>
+          <near>0.005</near>
+          <far>10</far>
+        </clip>
+        <camera_info_topic>/camera/camera_info</camera_info_topic>
+      </camera>
+    </sensor>
+  </gazebo>
+  <gazebo reference="lidar_link">
+    <sensor name="lidar" type="gpu_lidar">
+      <pose>0 0 0.006 0 0 0</pose>
+      <topic>/scan</topic>
+      <always_on>true</always_on>
+      <update_rate>10</update_rate>
+      <gz_frame_id>lidar_link</gz_frame_id>
+      <lidar>
+        <scan>
+          <horizontal>
+            <samples>720</samples>
+            <resolution>1</resolution>
+            <min_angle>-3.141592653589793</min_angle>
+            <max_angle>3.141592653589793</max_angle>
+          </horizontal>
+        </scan>
+        <range>
+          <min>0.03</min>
+          <max>5</max>
+          <resolution>0.005</resolution>
+        </range>
+      </lidar>
+    </sensor>
+  </gazebo>
+  <gazebo reference="base_link">
+    <sensor name="imu" type="imu">
+      <topic>/imu/data</topic>
+      <always_on>true</always_on>
+      <update_rate>50</update_rate>
+      <gz_frame_id>base_link</gz_frame_id>
+      <imu />
+    </sensor>
+  </gazebo>
   <gazebo>
     <plugin filename="gz-sim-diff-drive-system" name="gz::sim::systems::DiffDrive">
@@ -499,4 +558,30 @@
       <update_rate>50</update_rate>
     </plugin>
+    <plugin filename="gz-sim-wheel-slip-system" name="gz::sim::systems::WheelSlip">
+      <wheel link_name="wheel_left_link">
+        <wheel_radius>0.028</wheel_radius>
+        <wheel_normal_force>3.6836550000000003</wheel_normal_force>
+        <slip_compliance_lateral>0.5</slip_compliance_lateral>
+        <slip_compliance_longitudinal>0</slip_compliance_longitudinal>
+      </wheel>
+      <wheel link_name="wheel_left_front_link">
+        <wheel_radius>0.028</wheel_radius>
+        <wheel_normal_force>3.6836550000000003</wheel_normal_force>
+        <slip_compliance_lateral>0.5</slip_compliance_lateral>
+        <slip_compliance_longitudinal>0</slip_compliance_longitudinal>
+      </wheel>
+      <wheel link_name="wheel_right_link">
+        <wheel_radius>0.028</wheel_radius>
+        <wheel_normal_force>3.6836550000000003</wheel_normal_force>
+        <slip_compliance_lateral>0.5</slip_compliance_lateral>
+        <slip_compliance_longitudinal>0</slip_compliance_longitudinal>
+      </wheel>
+      <wheel link_name="wheel_right_front_link">
+        <wheel_radius>0.028</wheel_radius>
+        <wheel_normal_force>3.6836550000000003</wheel_normal_force>
+        <slip_compliance_lateral>0.5</slip_compliance_lateral>
+        <slip_compliance_longitudinal>0</slip_compliance_longitudinal>
+      </wheel>
+    </plugin>
   </gazebo>
 </robot>
