Commit message: 完整场景，速度修正，解决红绿灯问题。

File: src/dongfeng_description/urdf/dongfeng_car.urdf.xacro (robot description, xacro)
@@ -1,4 +1,6 @@
 <?xml version='1.0' encoding='utf-8'?>
-<robot name="dongfeng_car">
+<robot name="dongfeng_car" xmlns:xacro="http://www.ros.org/wiki/xacro">
+  <xacro:arg name="driving_mode" default="fast"/>
+  <xacro:property name="drive_limit" value="0.40"/>
   <!--Generated by scripts/generate_vehicle.py. X forward, Y left, Z up. Camera, lidar and IMU publish through Gazebo Sensors.-->
   <link name="base_link">
@@ -545,6 +547,6 @@
       <child_frame_id>base_link</child_frame_id>
       <odom_publish_frequency>50</odom_publish_frequency>
-      <min_linear_velocity>-0.25</min_linear_velocity>
-      <max_linear_velocity>0.25</max_linear_velocity>
+      <min_linear_velocity>-${drive_limit}</min_linear_velocity>
+      <max_linear_velocity>${drive_limit}</max_linear_velocity>
       <min_angular_velocity>-1.2</min_angular_velocity>
       <max_angular_velocity>1.2</max_angular_velocity>
